Commit message: A bit of tunning in the inertias and masses

File: robotiq_2f_model/model/inertias.urdf.xacro (robot description, xacro)
@@ -3,8 +3,8 @@
 <!-- length is along the z-axis! -->
 <xacro:macro name="cylinder_inertia" params="radius length mass">
-	<inertia ixx="${mass * (3 * radius * radius + length * length) / 12}" iyy="${mass * (3 * radius * radius + length * length) / 12}" izz="${mass * radius* radius / 2}" ixy="0" iyz="0" ixz="0"/>
+	<inertia ixx="${1000 * mass * (3 * radius * radius + length * length) / 12}" iyy="${1000 * mass * (3 * radius * radius + length * length) / 12}" izz="${1000 * mass * radius* radius / 2}" ixy="0" iyz="0" ixz="0"/>
 </xacro:macro>
 <xacro:macro name="box_inertia" params="x_dim y_dim z_dim mass">
-	<inertia ixx="${mass * (y_dim * y_dim + z_dim * z_dim) / 12}" iyy="${mass * (x_dim * x_dim + z_dim * z_dim) / 12}" izz="${mass * (x_dim * x_dim + y_dim * y_dim) / 12}" ixy="0" iyz="0" ixz="0"/>
+	<inertia ixx="${1000 * mass * (y_dim * y_dim + z_dim * z_dim) / 12}" iyy="${1000 * mass * (x_dim * x_dim + z_dim * z_dim) / 12}" izz="${1000 * mass * (x_dim * x_dim + y_dim * y_dim) / 12}" ixy="0" iyz="0" ixz="0"/>
 </xacro:macro>
 </robot>

File: robotiq_2f_model/model/robotiq_2f_85.urdf.xacro (robot description, xacro)
@@ -27,7 +27,7 @@
 		<link name="${name}_base">
 			<inertial>
-				<mass value="0.2"/>
+				<mass value="0.5"/>
 				<origin xyz="0 0 ${0.015*0.5}"  />
-				<cylinder_inertia radius="0.04" length="0.045" mass="0.2"/>
+				<cylinder_inertia radius="0.04" length="0.045" mass="0.5"/>
 			</inertial>
 			<visual>
@@ -47,5 +47,5 @@
 				<origin xyz="0 0 0.06" rpy="0 0 0"/>
 				<geometry>
-					<box size="0.03 0.04 0.06"/>
+					<box size="0.03 0.03 0.06"/>
 				</geometry>
 			</collision>
@@ -69,7 +69,7 @@
 		<link name="${name}_right_driver">
 			<inertial>
-				<mass value="0.05"/>
+				<mass value="0.1"/>
 				<origin xyz="0 0.02 0" rpy="0 0 0" />
-				<box_inertia x_dim="0.02" y_dim="0.04" z_dim="0.02" mass="0.05"/>
+				<box_inertia x_dim="0.02" y_dim="0.04" z_dim="0.02" mass="0.1"/>
 			</inertial>
 			<visual>
@@ -80,7 +80,7 @@
 			<xacro:unless value="${precise_collision}">
 			<collision>
-				<origin xyz="0 0.02 0" rpy="-0.1 0 0"/>
-				<geometry>
-					<box size="0.02 0.04 0.02"/>
+				<origin xyz="0 0.01 0" rpy="-0.1 0 0"/>
+				<geometry>
+					<box size="0.002 0.004 0.002"/>
 				</geometry>
 			</collision>
@@ -112,7 +112,7 @@
 		<link name="${name}_right_coupler">
 			<inertial>
-				<mass value="0.05"/>
+				<mass value="0.1"/>
 				<origin xyz="0 0.0 0.025" rpy="-1.7 0 0"/>
-				<box_inertia x_dim="0.03" y_dim="0.065" z_dim="0.02" mass="0.05"/>
+				<box_inertia x_dim="0.03" y_dim="0.065" z_dim="0.02" mass="0.1"/>
 			</inertial>
 			<visual>
@@ -149,7 +149,7 @@
 		<link name="${name}_right_follower">
 			<inertial>
-				<mass value="0.05"/>
+				<mass value="0.1"/>
 				<origin xyz="0 -0.018 0.022" />
-				<box_inertia x_dim="0.02" y_dim="0.015" z_dim="0.048" mass="0.05"/>
+				<box_inertia x_dim="0.02" y_dim="0.015" z_dim="0.048" mass="0.1"/>
 			</inertial>
 			<visual>
@@ -160,7 +160,7 @@
 			<xacro:unless value="${precise_collision}">
 			<collision>
-				<origin xyz="0 -0.018 0.022" rpy="0 0 0"/>
-				<geometry>
-					<box size="0.02 0.015 0.048"/>
+				<origin xyz="0 -0.01 0.022" rpy="0 0 0"/>
+				<geometry>
+					<box size="0.002 0.0015 0.0048"/>
 				</geometry>
 			</collision>
@@ -181,7 +181,7 @@
 			<link name="${name}_right_pad">
 				<inertial>
-					<mass value="0.01"/>
+					<mass value="0.1"/>
 					<origin xyz="0 -0.022 0.031" />
-					<box_inertia x_dim="0.02" y_dim="0.008" z_dim="0.036" mass="0.01"/>
+					<box_inertia x_dim="0.02" y_dim="0.008" z_dim="0.036" mass="0.1"/>
 				</inertial>
 				<visual>
@@ -219,7 +219,7 @@
 		<link name="${name}_right_spring_link">
 			<inertial>
-				<mass value="0.05"/>
+				<mass value="0.1"/>
 				<origin xyz="0 0.018 0.018" rpy="-0.7068 0 0"/>
-				<box_inertia x_dim="0.04" y_dim="0.02" z_dim="0.065" mass="0.05"/>
+				<box_inertia x_dim="0.04" y_dim="0.02" z_dim="0.065" mass="0.1"/>
 			</inertial>
 			<visual>
@@ -230,7 +230,7 @@
 			<xacro:unless value="${precise_collision}">
 			<collision>
-				<origin xyz="0 0.018 0.018" rpy="-0.7068 0 0"/>
-				<geometry>
-					<box size="0.04 0.02 0.065"/>
+				<origin xyz="0 0.025 0.015" rpy="-0.7068 0 0"/>
+				<geometry>
+					<box size="0.004 0.002 0.0065"/>
 				</geometry>
 			</collision>
@@ -257,7 +257,7 @@
 		<link name="${name}_left_driver">
 			<inertial>
-				<mass value="0.05"/>
+				<mass value="0.1"/>
 				<origin xyz="0 0.02 0" rpy="0 0 0" />
-				<box_inertia x_dim="0.02" y_dim="0.04" z_dim="0.02" mass="0.05"/>
+				<box_inertia x_dim="0.02" y_dim="0.04" z_dim="0.02" mass="0.1"/>
 			</inertial>
 			<visual>
@@ -268,7 +268,7 @@
 			<xacro:unless value="${precise_collision}">
 			<collision>
-				<origin xyz="0 0.02 0" rpy="-0.1 0 0"/>
-				<geometry>
-					<box size="0.02 0.04 0.02"/>
+				<origin xyz="0 0.01 0" rpy="-0.1 0 0"/>
+				<geometry>
+					<box size="0.002 0.004 0.002"/>
 				</geometry>
 			</collision>
@@ -300,7 +300,7 @@
 		<link name="${name}_left_coupler">
 			<inertial>
-				<mass value="0.05"/>
+				<mass value="0.1"/>
 				<origin xyz="0 0.0 0.025" rpy="-1.7 0 0"/>
-				<box_inertia x_dim="0.03" y_dim="0.065" z_dim="0.02" mass="0.05"/>
+				<box_inertia x_dim="0.03" y_dim="0.065" z_dim="0.02" mass="0.1"/>
 			</inertial>
 			<visual>
@@ -337,7 +337,7 @@
 		<link name="${name}_left_follower">
 			<inertial>
-				<mass value="0.05"/>
+				<mass value="0.1"/>
 				<origin xyz="0 -0.018 0.022" />
-				<box_inertia x_dim="0.02" y_dim="0.015" z_dim="0.048" mass="0.05"/>
+				<box_inertia x_dim="0.02" y_dim="0.015" z_dim="0.048" mass="0.1"/>
 			</inertial>
 			<visual>
@@ -348,7 +348,7 @@
 			<xacro:unless value="${precise_collision}">
 			<collision>
-				<origin xyz="0 -0.018 0.022" rpy="0 0 0"/>
-				<geometry>
-					<box size="0.02 0.015 0.048"/>
+				<origin xyz="0 -0.01 0.022" rpy="0 0 0"/>
+				<geometry>
+					<box size="0.002 0.0015 0.0048"/>
 				</geometry>
 			</collision>
@@ -369,7 +369,7 @@
 			<link name="${name}_left_pad">
 				<inertial>
-					<mass value="0.01"/>
+					<mass value="0.1"/>
 					<origin xyz="0 -0.022 0.031" />
-					<box_inertia x_dim="0.02" y_dim="0.008" z_dim="0.036" mass="0.01"/>
+					<box_inertia x_dim="0.02" y_dim="0.008" z_dim="0.036" mass="0.1"/>
 				</inertial>
 				<visual>
@@ -407,7 +407,7 @@
 		<link name="${name}_left_spring_link">
 			<inertial>
-				<mass value="0.05"/>
+				<mass value="0.1"/>
 				<origin xyz="0 0.018 0.018" rpy="-0.7068 0 0"/>
-				<box_inertia x_dim="0.04" y_dim="0.02" z_dim="0.065" mass="0.05"/>
+				<box_inertia x_dim="0.04" y_dim="0.02" z_dim="0.065" mass="0.1"/>
 			</inertial>
 			<visual>
@@ -418,7 +418,7 @@
 			<xacro:unless value="${precise_collision}">
 			<collision>
-				<origin xyz="0 0.018 0.018" rpy="-0.7068 0 0"/>
-				<geometry>
-					<box size="0.04 0.02 0.065"/>
+				<origin xyz="0 0.025 0.015" rpy="-0.7068 0 0"/>
+				<geometry>
+					<box size="0.004 0.002 0.0065"/>
 				</geometry>
 			</collision>

File: robotiq_2f_model/model/robotiq_ur_coupler.urdf.xacro (robot description, xacro)
@@ -5,5 +5,5 @@
 	<joint name="${name}_coupler_joint" type="fixed">
 		<!-- total height of coupler, minus the depth of robot end-effector shape and the gripper small depth-->
-		<origin xyz="0 0 ${0.001*(13.9-3-3)}" rpy="0 0 0" />
+		<origin xyz="0 0 ${0.001*(13.5-3-3)}" rpy="0 0 0" />
 		<parent link="${parent}"/>
 		<child link="${name}"/>
@@ -11,5 +11,5 @@
 	<link name="${name}">
 		<visual>
-			<origin xyz="0 0 ${-1*0.001*(13.9-3-3)*0.5}" rpy="0 0 0" />
+			<origin xyz="0 0 ${-1*0.001*(13.93-3)*0.5}" rpy="0 0 0" />
 			<geometry>
 				<!-- only the visible part of the coupler -->
@@ -23,11 +23,11 @@
 			<origin xyz="0 0 0" rpy="0 0 0" />
 			<geometry>
-				<cylinder length="${0.001*(13.9)}" radius="${0.5*0.075}" />
+				<cylinder length="${0.001*(13.5)}" radius="${0.5*0.075}" />
 			</geometry>
 		</collision>
 		<inertial>
-			<mass value="0.1"/>
+			<mass value="0.3"/>
 			<origin xyz="0 0 ${0.001*(13.9)*0.5}"  />
-			<cylinder_inertia radius="${0.5*0.075}" length="${0.001*(13.9)}" mass="0.1"/>
+			<cylinder_inertia radius="${0.5*0.075}" length="${0.001*(13.9)}" mass="0.3"/>
 		</inertial>
 	</link>
